File: turnstileUHF/_autosave-turnstileUHF.kicad_sch (KiCad schematic)
At the start: 37 parts, among them Q1 PMOS, SW1 SW_DIP_x01

Commit message: burn wire circuit
Parts:
- removed C1: C_Small, symbol Device:C_Small
- removed Q1: PMOS, symbol Simulation_SPICE:PMOS
- removed R_Load: R, symbol Device:R
- removed SW1: SW_DIP_x01, symbol Switch:SW_DIP_x01
- added Q1, Q2, Q3, Q4, Q8: 2N7002, Package_TO_SOT_SMD:SOT-23, symbol Transistor_FET:2N7002
- added Q5, Q6, Q7: AO3401A, Package_TO_SOT_SMD:SOT-23, symbol Transistor_FET:AO3401A
- added R2, R3, R4: R_burn, symbol Device:R
- added R_Pulldown1, R_Pulldown2, R_Pulldown3, R_Pulldown4: 10k, symbol Device:R
- added SW1: SW_DIP_x04, symbol Switch:SW_DIP_x04
- R1: value 100k -> R_burn
Connections:
- net +8V: now also SW1.1, SW1.2, SW1.3, SW1.4
- net GND: now also R1.2, Q1.2 (S), Q2.2 (S), Q3.2 (S), R2.2, R3.2
- net at R1.1: now also Q5.3 (D)
- new net: Q8.1 (G), R_Pulldown4.1, SW1.8
- new net: Q4.2 (S), R_Pulldown4.2
- new net: Q7.3 (D), R3.1
- new net: Q1.3 (D), Q5.1 (G)
- new net: Q5.2 (S), R_Pulldown1.2
- new net: Q6.3 (D), R2.1
- new net: Q1.1 (G), R_Pulldown1.1, SW1.5
- new net: Q3.1 (G), R_Pulldown3.1, SW1.7
- new net: Q7.2 (S), R_Pulldown3.2
- new net: Q2.1 (G), R_Pulldown2.1, SW1.6
- new net: Q2.3 (D), Q6.1 (G)
- new net: Q6.2 (S), R_Pulldown2.2
- new net: Q4.1 (G), Q8.3 (D)
- new net: Q3.3 (D), Q7.1 (G)
