File: turnstileUHF/turnstileUHF.kicad_pcb (KiCad board)
At the start: 2 copper layers, 98 x 98 mm, 53 parts, among them J5 RFPC-SMA28-F, Q1 2N7002, Q2 2N7002, Q3 2N7002, Q4 2N7002, Q5 AO3401A, Q6 AO3401A, Q7 AO3401A, Q8 2N7002, U1 74HCT238D

Commit message: Changes made to keep out zones to allow antenna traces
Routing:
- net Net-(ANT2-~): track 0.00 -> 35.2 mm
Changed lines of the file:
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@@
+	)
+	(segment
+		(start 177 128.092102)
+		(end 166.092102 139)
+		(width 0.2)
+		(layer "F.Cu")
+		(net "Net-(ANT2-~)")
+	)
+	(segment
+		(start 166 139)
+		(end 166 141.5)
+		(width 0.2)
+		(layer "F.Cu")
+		(net "Net-(ANT2-~)")
+	)
+	(segment
+		(start 166 141.5)
+		(end 170.5 146)
+		(width 0.2)
+		(layer "F.Cu")
+		(net "Net-(ANT2-~)")
+	)
+	(segment
+		(start 166.092102 139)
+		(end 166 139)
+		(width 0.2)
+		(layer "F.Cu")
+		(net "Net-(ANT2-~)")
+	)
+	(segment
+		(start 170.5 146)
+		(end 170.5 156.849999)
+		(width 0.2)
+		(layer "F.Cu")
+		(net "Net-(ANT2-~)")
 	)
 	(segment
@@
 		(min_thickness 0.25)
 		(keepout
-			(tracks not_allowed)
+			(tracks allowed)
 			(vias not_allowed)
 			(pads allowed)
@@
 		(min_thickness 0.25)
 		(keepout
-			(tracks not_allowed)
+			(tracks allowed)
 			(vias not_allowed)
 			(pads allowed)
@@
 		(min_thickness 0.25)
 		(keepout
-			(tracks not_allowed)
+			(tracks allowed)
 			(vias not_allowed)
 			(pads allowed)
@@
 		(min_thickness 0.25)
 		(keepout
-			(tracks not_allowed)
-			(vias not_allowed)
-			(pads allowed)
+			(tracks allowed)
+			(vias not_allowed)
+			(pads allowed)

Commit message: added missing antenna trace
Parts:
- added ANT1: Antenna, RF_Antenna:Coilcraft_MA5532-AE_RFID, F.Cu at (190.9, 98.7)
Routing:
- net Net-(ANT1-~): track 35.2 -> 30.7 mm
