File: doorsensing/doorsensing.kicad_sch (KiCad schematic)
At the start: 2 parts, among them U1 ADS1115IDGSR, U2 OPA333xxD

Commit message: continued working schematic
Parts:
- added C1, C2: C, symbol Device:C
- added R1, R10, R2, R3, R4, R5, R6, R7, R8, R9: R_US, symbol Device:R_US
Connections:
- net GND: now also U1.1 (ADDR), U1.3 (GND), U1.6 (AIN2), U1.7 (AIN3), U2.4 (V-), C1.2, C2.1
- net at U1.10 (SCL): now also R4.2
- net at U1.5 (AIN1): now also R3.1
- net VDD: now reaches U1.8 (VDD)
- net VDD: now also U2.7 (V+), C2.2, R2.1, R3.2, R4.1, R5.1
- net at U1.9 (SDA): now also R5.2
- net at U2.3 (+): now also C1.1, R1.2
- new net: R1.1, R2.2, R6.1, R7.1, R8.1, R9.1
- no-connect marks 0 -> 1

Commit message: first iteration of schematic done
Parts:
- added C3: 100 nF, symbol Device:C
- added J1, J3: Conn_01x02, symbol Connector_Generic:Conn_01x02
- added J2: Conn_01x04, symbol Connector_Generic:Conn_01x04
- added SW1, SW2, SW3, SW4: SW_SPST, symbol Switch:SW_SPST
- added U3: TPD1E05U06DYA, Diode_SMD:D_SOD-523, symbol Power_Protection:TPD1E05U06DYA
- C1: value C -> 10 nF
- C2: value C -> 100 nF
- R1: value R_US -> 11k
- R10, R6: value R_US -> 1M
- R2: value R_US -> 64.9k
- R3: value R_US -> 31k
- R4: value R_US -> 4.7k
- R5: value R_US -> 4.79k
- R7: value R_US -> 499k
- R8: value R_US -> 249k
- R9: value R_US -> 124k
Connections:
- net GND: now also C3.2, J2.2 (Pin_2), J3.1 (Pin_1), U3.2 (GND)
- net VDD: now also C3.1, J2.1 (Pin_1), J2.3 (Pin_3), J2.4 (Pin_4)
- net sense: now reaches R1.1, R2.2, R6.1, R7.1, R8.1, R9.1
- net sense: now also R10.1, J1.2 (Pin_2), J3.2 (Pin_2), U3.1 (I/O)
- net at R8.2: now also SW3.1 (A)
- net at R6.2: now also SW1.1 (A)
- net at R7.2: now also SW2.1 (A)
- net at R9.2: now also SW4.1 (A)
- net at R10.2: now also J1.1 (Pin_1), SW1.2 (B), SW2.2 (B), SW3.2 (B), SW4.2 (B)
Other:
- note added: "I/O Flight Controller"
- note added: "Inside"
- note added: "Outside/ Doors"

Commit message: made revision after review 1
Parts:
- C1, C2, C3: footprint (none) -> Capacitor_SMD:C_0603_1608Metric
- J1, J3: footprint (none) -> Connector_JST:JST_PH_S2B-PH-K_1x02_P2.00mm_Horizontal
- J2: footprint (none) -> Connector_JST:JST_PH_S4B-PH-K_1x04_P2.00mm_Horizontal
- R1: value 11k -> 1k; footprint (none) -> Resistor_SMD:R_0603_1608Metric
- R10, R2, R6, R7, R8, R9: footprint (none) -> Resistor_SMD:R_0603_1608Metric
- R3: value 31k -> 1k; footprint (none) -> Resistor_SMD:R_0603_1608Metric
- R4: footprint (none) -> Resistor_SMD:R_0603_1608Metric; now not fitted
- R5: value 4.79k -> 4.7k; footprint (none) -> Resistor_SMD:R_0603_1608Metric; now not fitted
- U1: value ADS1115IDGSR -> ADS1015IDGSR; MPN (none) -> ADS1015IDGSR
Connections:
- net at R4.2, U1.10 (SCL): now also J2.4 (Pin_4)
- net at R5.2, U1.9 (SDA): now also J2.3 (Pin_3)
- net VDD renamed 3.3V
- net 3.3V: no longer J2.3 (Pin_3), J2.4 (Pin_4)
Other:
- note added: "The PU resistors will be on the flight controller. Only include resistor for testing"
- note added: "switches placeholder for door contact pads"
